Commit message: smooth turns are faster; added forward correction when there is a front wall; wheels moved to the back

File: micromouse_description/urdf/mouse.xacro (robot description, xacro)
@@ -8,5 +8,5 @@
   <xacro:property name="wheel_thickness" value="0.005"/>
   <xacro:property name="base_wheel_gap" value="${wheel_thickness/2}"/>
-  <xacro:property name="wheel_joint_offset" value="0.01"/>
+  <xacro:property name="wheel_joint_offset" value="-0.01"/>
   <xacro:property name="caster_wheel_radius" value="0.005"/>
   <xacro:property name="caster_wheel_mass" value="0.001"/>
@@ -65,5 +65,5 @@
 <link name="back_caster_link">
 <visual>
-      <origin xyz="-${caster_wheel_offset} 0 -${base_thickness/2+caster_wheel_radius}" rpy="0 0 0"/>
+      <origin xyz="${caster_wheel_offset} 0 -${base_thickness/2+caster_wheel_radius}" rpy="0 0 0"/>
       <geometry>
 	<sphere radius="${caster_wheel_radius}"/>
@@ -72,5 +72,5 @@
     </visual>
     <collision>
-      <origin xyz="-${caster_wheel_offset} 0 -${base_thickness/2+caster_wheel_radius}" rpy="0 0 0"/>
+      <origin xyz="${caster_wheel_offset} 0 -${base_thickness/2+caster_wheel_radius}" rpy="0 0 0"/>
       <geometry>
         <sphere radius="${caster_wheel_radius}"/>

Commit message: major changes: mouse description looks like a DC mouse; added top view camera mode in gazebo; added accelerations and decelerations

File: micromouse_description/urdf/mouse.xacro (robot description, xacro)
@@ -1,22 +1,26 @@
 <?xml version="1.0"?>
 <robot xmlns:xacro="http://www.ros.org/wiki/xacro" name="vayu">
-  <xacro:property name="base_width" value="0.07"/>
-  <xacro:property name="base_len" value="0.07"/>
-  <xacro:property name="base_thickness" value="0.02"/>
+  <xacro:property name="mouse_width" value="0.075"/>
+  <xacro:property name="mouse_len" value="0.10"/>
+  <xacro:property name="base_width" value="${mouse_width-2*wheel_thickness-2*base_wheel_gap}"/>
+  <xacro:property name="base_len" value="${2*wheel_radius}"/>
+  <xacro:property name="base_thickness" value="0.005"/>
+  <xacro:property name="base_wheel_gap" value="${0.001}"/>
+  <xacro:property name="base_curve_radius" value="0.03"/>
+  <xacro:property name="base_zoffset" value="${(wheel_radius-caster_wheel_radius*2-base_thickness/2)}"/>
   <xacro:property name="wheel_radius" value="0.02"/>
-  <xacro:property name="wheel_separation" value="${(base_width+2*base_wheel_gap)}"/>
-  <xacro:property name="wheel_thickness" value="0.005"/>
-  <xacro:property name="base_wheel_gap" value="${wheel_thickness/2}"/>
+  <xacro:property name="wheel_separation" value="${(base_width+2*base_wheel_gap+wheel_thickness)}"/>
+  <xacro:property name="wheel_thickness" value="0.01"/>
   <xacro:property name="wheel_joint_offset" value="-0.01"/>
   <xacro:property name="caster_wheel_radius" value="0.005"/>
   <xacro:property name="caster_wheel_mass" value="0.001"/>
-  <xacro:property name="caster_wheel_offset" value="${base_len/2-caster_wheel_radius}"/>
+  <xacro:property name="caster_wheel_offset" value="${mouse_len+wheel_joint_offset-base_len/2-caster_wheel_radius}"/>
   <xacro:property name="caster_support_length" value="${wheel_radius-base_thickness/2-2*caster_wheel_radius-0.001}"/>
-  <xacro:property name="laser_size_x" value="0.01"/>
-  <xacro:property name="laser_size_y" value="0.01"/>
-  <xacro:property name="laser_size_z" value="0.01"/>
-  <xacro:property name="laser_origin_x" value="${base_len/2}"/>
+  <xacro:property name="laser_size_x" value="0.005"/>
+  <xacro:property name="laser_size_y" value="0.005"/>
+  <xacro:property name="laser_size_z" value="0.005"/>
+  <xacro:property name="laser_origin_x" value="${mouse_len+wheel_joint_offset-base_len/2-laser_size_x/2}"/>
   <xacro:property name="laser_origin_y" value="0"/>
-  <xacro:property name="laser_origin_z" value="0"/>
+  <xacro:property name="laser_origin_z" value="-${base_zoffset-base_thickness/2-laser_size_z/2}"/>
   <!--Color Properties-->
   <material name="blue">
@@ -42,4 +46,5 @@
   <link name="base_link">
     <visual>
+      <origin xyz="${wheel_joint_offset} 0 -${base_zoffset}" rpy="0 0 0"/>
       <geometry>
         <box size="${base_len} ${base_width} ${base_thickness}"/>
@@ -47,8 +52,65 @@
       <material name="green"/>
     </visual>
+    <visual>
+      <origin xyz="${wheel_joint_offset+base_len/2+(mouse_len-base_len-base_curve_radius)/2} 0 -${base_zoffset}" rpy="0 0 0"/>
+      <geometry>
+        <box size="${(mouse_len-base_len-base_curve_radius)} ${mouse_width} ${base_thickness}"/>
+      </geometry>
+      <material name="green"/>
+    </visual>
+    <visual>
+      <origin xyz="${wheel_joint_offset+base_len/2+(mouse_len-base_len-base_curve_radius)} ${mouse_width/2-base_curve_radius} -${base_zoffset}" rpy="0 0 0"/>
+      <geometry>
+        <cylinder radius="${base_curve_radius}" length="${base_thickness}"/>
+      </geometry>
+      <material name="green"/>
+    </visual>
+    <visual>
+      <origin xyz="${wheel_joint_offset+base_len/2+(mouse_len-base_len-base_curve_radius)} -${mouse_width/2-base_curve_radius} -${base_zoffset}" rpy="0 0 0"/>
+      <geometry>
+        <cylinder radius="${base_curve_radius}" length="${base_thickness}"/>
+      </geometry>
+      <material name="green"/>
+    </visual>
+    <visual>
+      <origin xyz="${wheel_joint_offset+base_len/2+mouse_len-base_len-base_curve_radius/2} 0 -${base_zoffset}" rpy="0 0 0"/>
+      <geometry>
+        <box size="${base_curve_radius} ${mouse_width-2*base_curve_radius} ${base_thickness}"/>
+      </geometry>
+      <material name="green"/>
+    </visual>
     <collision name="base_collision">
+      <origin xyz="${wheel_joint_offset} 0 -${base_zoffset}" rpy="0 0 0"/>
       <geometry>
         <box size="${base_len} ${base_width} ${base_thickness}"/>
       </geometry>
+    </collision>
+    <collision name="base_1_collision">
+      <origin xyz="${wheel_joint_offset+base_len/2+(mouse_len-base_len-base_curve_radius)/2} 0 -${base_zoffset}" rpy="0 0 0"/>
+      <geometry>
+        <box size="${(mouse_len-base_len-base_curve_radius)} ${mouse_width} ${base_thickness}"/>
+      </geometry>
+      <material name="green"/>
+    </collision>
+    <collision name="base_2_collision">
+      <origin xyz="${wheel_joint_offset+base_len/2+(mouse_len-base_len-base_curve_radius)} ${mouse_width/2-base_curve_radius} -${base_zoffset}" rpy="0 0 0"/>
+      <geometry>
+        <cylinder radius="${base_curve_radius}" length="${base_thickness}"/>
+      </geometry>
+      <material name="green"/>
+    </collision>
+    <collision name="base_3_collision">
+      <origin xyz="${wheel_joint_offset+base_len/2+(mouse_len-base_len-base_curve_radius)} -${mouse_width/2-base_curve_radius} -${base_zoffset}" rpy="0 0 0"/>
+      <geometry>
+        <cylinder radius="${base_curve_radius}" length="${base_thickness}"/>
+      </geometry>
+      <material name="green"/>
+    </collision>
+    <collision name="base_4_collision">
+      <origin xyz="${wheel_joint_offset+base_len/2+mouse_len-base_len-base_curve_radius/2} 0 -${base_zoffset}" rpy="0 0 0"/>
+      <geometry>
+        <box size="${base_curve_radius} ${mouse_width-2*base_curve_radius} ${base_thickness}"/>
+      </geometry>
+      <material name="green"/>
     </collision>
     <inertial>
@@ -59,11 +121,25 @@
   <!--base_link to base_footprint Joint-->
   <joint name="base_link_joint" type="fixed">
-    <origin xyz="0 0 ${wheel_radius + 0.005}" rpy="0 0 0" />
+    <origin xyz="0 0 ${wheel_radius}" rpy="0 0 0" />
     <parent link="base_footprint"/>
     <child link="base_link" />
   </joint>
+  <link name="circuit_link">
+    <visual>
+      <origin xyz="0 0 0" rpy="0 0 0" />
+      <geometry>
+        <box size="${mouse_len/4} ${mouse_width/3} 0.001"/>
+      </geometry>
+      <material name="black"/>
+    </visual>
+  </link>
+  <joint name="circuit_joint" type="fixed">
+    <origin xyz="${wheel_joint_offset+base_len/2+(mouse_len-base_len-base_curve_radius)/2} 0 -${base_zoffset-base_thickness/2}" rpy="0 0 0" />
+    <parent link="base_link"/>
+    <child link="circuit_link" />
+  </joint>
 <link name="back_caster_link">
 <visual>
-      <origin xyz="${caster_wheel_offset} 0 -${base_thickness/2+caster_wheel_radius}" rpy="0 0 0"/>
+      <origin xyz="${caster_wheel_offset} 0 -${base_zoffset+base_thickness/2+caster_wheel_radius}" rpy="0 0 0"/>
       <geometry>
 	<sphere radius="${caster_wheel_radius}"/>
@@ -72,5 +148,5 @@
     </visual>
     <collision>
-      <origin xyz="${caster_wheel_offset} 0 -${base_thickness/2+caster_wheel_radius}" rpy="0 0 0"/>
+      <origin xyz="${caster_wheel_offset} 0 -${base_zoffset+base_thickness/2+caster_wheel_radius}" rpy="0 0 0"/>
       <geometry>
         <sphere radius="${caster_wheel_radius}"/>
@@ -83,24 +159,4 @@
     <child link="back_caster_link" />
   </joint>
-<!--link name="front_caster_link">
-<visual>
-      <origin xyz="${caster_wheel_offset} 0 -${base_thickness/2+caster_wheel_radius}" rpy="0 0 0"/>
-      <geometry>
-	<sphere radius="${caster_wheel_radius}"/>
-      </geometry>
-      <material name="black"/>
-    </visual>
-    <collision>
-      <origin xyz="${caster_wheel_offset} 0 -${base_thickness/2+caster_wheel_radius}" rpy="0 0 0"/>
-      <geometry>
-        <sphere radius="${caster_wheel_radius}"/>
-      </geometry>
-    </collision>
-</link>
-  <joint name="front_caster_link_joint" type="fixed">
-    <origin xyz="0 0 0" rpy="0 0 0" />
-    <parent link="base_link"/>
-    <child link="front_caster_link" />
-  </joint-->
   <!--Wheel link & joint macro-->
   <xacro:macro name="wheel" params="prefix reflect">
@@ -128,5 +184,5 @@
       <parent link="base_link"/>
       <child link="${prefix}_wheel"/>
-      <origin xyz="${wheel_joint_offset} ${((base_width/2)+base_wheel_gap)*reflect} 0" rpy="0 0 0"/>
+      <origin xyz="${wheel_joint_offset} ${((base_width/2)+base_wheel_gap+wheel_thickness/2)*reflect} 0" rpy="0 0 0"/>
 <limit effort="100" velocity="100"/>
       <joint_properties damping="0.0" friction="0.0"/>
@@ -136,4 +192,29 @@
   <xacro:wheel prefix="left" reflect="1"/>
   <xacro:wheel prefix="right" reflect="-1"/>
+  <!--Motor link & joint macro-->
+  <xacro:macro name="motor" params="prefix reflect">
+    <link name="${prefix}_motor">
+      <visual>
+        <geometry>
+          <cylinder radius="${wheel_radius-base_zoffset-base_thickness/2}" length="${base_width/2-base_wheel_gap}"/>
+        </geometry>
+        <material name="grey"/>
+      </visual>
+      <collision>
+        <geometry>
+          <cylinder radius="${wheel_radius-base_zoffset-base_thickness/2}" length="${wheel_thickness}"/>
+        </geometry>
+      </collision>
+    </link>
+    <joint name="${prefix}_motor_joint" type="fixed">
+      <origin xyz="0 ${((base_width/2-0.005)/2+base_wheel_gap)*reflect} 0" rpy="${pi/2} 0 0"/>
+      <parent link="${prefix}_wheel"/>
+      <child link="${prefix}_motor"/>
+      <origin xyz="0 0 0" rpy="0 0 0"/>
+    </joint>
+  </xacro:macro>
+  <!--Create Left & Right Wheel links/joints-->
+  <xacro:motor prefix="left" reflect="-1"/>
+  <xacro:motor prefix="right" reflect="1"/>
   <!--Create Left & Right Wheel links/joints-->
   <!--Laser-->

File: micromouse_description/urdf/mouse_gazebo.xacro (robot description, xacro)
@@ -42,4 +42,31 @@
               <minDepth>0</minDepth>
   </gazebo>
+  <gazebo reference="circuit_link">
+    <material>Gazebo/Black</material>
+              <mu1>10</mu1>
+              <mu2>10</mu2>
+              <kp>1000000.0</kp>
+              <kd>100.0</kd>
+              <maxVel>0.01</maxVel>
+              <minDepth>0</minDepth>
+  </gazebo>
+  <gazebo reference="left_motor">
+    <material>Gazebo/Grey</material>
+              <mu1>10</mu1>
+              <mu2>10</mu2>
+              <kp>1000000.0</kp>
+              <kd>100.0</kd>
+              <maxVel>0.01</maxVel>
+              <minDepth>0</minDepth>
+  </gazebo>
+  <gazebo reference="right_motor">
+    <material>Gazebo/Grey</material>
+              <mu1>10</mu1>
+              <mu2>10</mu2>
+              <kp>1000000.0</kp>
+              <kd>100.0</kd>
+              <maxVel>0.01</maxVel>
+              <minDepth>0</minDepth>
+  </gazebo>
   <gazebo reference="base_link">
     <material>Gazebo/Green</material>
@@ -56,5 +83,5 @@
       <alwaysOn>false</alwaysOn>
       <legacyMode>false</legacyMode>
-      <updateRate>30</updateRate>
+      <updateRate>100</updateRate>
       <leftJoint>left_wheel_joint</leftJoint>
       <rightJoint>right_wheel_joint</rightJoint>
@@ -62,6 +89,6 @@
       <wheelDiameter>${wheel_radius * 2}</wheelDiameter>
       <torque>20</torque>
-      <commandTopic>/kbot/base_controller/cmd_vel</commandTopic>
-      <odometryTopic>/kbot/base_controller/odom</odometryTopic>
+      <commandTopic>cmd_vel</commandTopic>
+      <odometryTopic>odom</odometryTopic>
       <odometryFrame>odom</odometryFrame>
       <robotBaseFrame>base_footprint</robotBaseFrame>
@@ -72,6 +99,6 @@
     <sensor type="ray" name="head_hokuyo_sensor">
       <pose>0 0 0 0 0 0</pose>
-      <visualize>true</visualize>
-      <update_rate>20</update_rate>
+      <visualize>false</visualize>
+      <update_rate>100</update_rate>
       <ray>
         <scan>
@@ -85,5 +112,5 @@
         <range>
           <min>0.01</min>
-          <max>2</max>
+          <max>1</max>
           <resolution>0.005</resolution>
         </range>
@@ -95,5 +122,5 @@
       </ray>
       <plugin name="gazebo_ros_head_hokuyo_controller" filename="libgazebo_ros_laser.so">
-        <topicName>/kbot/laser_scan/scan</topicName>
+        <topicName>scan</topicName>
         <frameName>sensor_laser</frameName>
       </plugin>

Commit message: minor changes to the model

File: micromouse_description/urdf/mouse.xacro (robot description, xacro)
@@ -7,7 +7,7 @@
   <xacro:property name="base_thickness" value="0.005"/>
   <xacro:property name="base_wheel_gap" value="${0.001}"/>
-  <xacro:property name="base_curve_radius" value="0.03"/>
+  <xacro:property name="base_curve_radius" value="0.029"/>
   <xacro:property name="base_zoffset" value="${(wheel_radius-caster_wheel_radius*2-base_thickness/2)}"/>
-  <xacro:property name="wheel_radius" value="0.02"/>
+  <xacro:property name="wheel_radius" value="0.025"/>
   <xacro:property name="wheel_separation" value="${(base_width+2*base_wheel_gap+wheel_thickness)}"/>
   <xacro:property name="wheel_thickness" value="0.01"/>
@@ -20,5 +20,5 @@
   <xacro:property name="laser_size_y" value="0.005"/>
   <xacro:property name="laser_size_z" value="0.005"/>
-  <xacro:property name="laser_origin_x" value="${mouse_len+wheel_joint_offset-base_len/2-laser_size_x/2}"/>
+  <xacro:property name="laser_origin_x" value="${mouse_len+wheel_joint_offset-base_len/2-laser_size_x/2-0.015}"/>
   <xacro:property name="laser_origin_y" value="0"/>
   <xacro:property name="laser_origin_z" value="-${base_zoffset-base_thickness/2-laser_size_z/2}"/>

File: micromouse_description/urdf/mouse_gazebo.xacro (robot description, xacro)
@@ -79,9 +79,26 @@
               <minDepth>0</minDepth>
   </gazebo>
+  <gazebo reference="led">
+ <material>
+            <ambient>1 0.2 0.2 1</ambient>
+            <diffuse>1 0.2 0.2 1</diffuse>
+            <specular>1 1 1 1</specular>
+            <emissive>1 0.2 0.2 1</emissive>
+          </material>
+        <light name='button' type='point'>
+          <pose>0 0 0.05 0 0 0</pose>
+          <attenuation>
+            <range>0.02</range>
+            <linear>0.10</linear>
+          </attenuation>
+          <diffuse>1 0.2 0.2 1</diffuse>
+          <specular>1 1 1 1</specular>
+        </light>
+  </gazebo>
   <gazebo>
     <plugin name="differential_drive_controller" filename="libgazebo_ros_diff_drive.so">
       <alwaysOn>false</alwaysOn>
       <legacyMode>false</legacyMode>
-      <updateRate>100</updateRate>
+      <updateRate>200</updateRate>
       <leftJoint>left_wheel_joint</leftJoint>
       <rightJoint>right_wheel_joint</rightJoint>
@@ -99,6 +116,6 @@
     <sensor type="ray" name="head_hokuyo_sensor">
       <pose>0 0 0 0 0 0</pose>
-      <visualize>false</visualize>
-      <update_rate>100</update_rate>
+      <visualize>true</visualize>
+      <update_rate>200</update_rate>
       <ray>
         <scan>
@@ -112,5 +129,5 @@
         <range>
           <min>0.01</min>
-          <max>1</max>
+          <max>0.25</max>
           <resolution>0.005</resolution>
         </range>
