Commit message: changed led shape to look like leds

File: micromouse_description/urdf/mouse.xacro (robot description, xacro)
@@ -39,4 +39,7 @@
     <color rgba="0.1 0.7 0.1 1"/>
   </material>
+  <material name="darkgrey">
+    <color rgba="0.1 0.1 0.1 1"/>
+  </material>
   <!--Base Footprint-->
   <link name="base_footprint">
@@ -114,8 +117,4 @@
       <material name="green"/>
     </collision>
-    <inertial>
-      <mass value="5"/>
-      <inertia ixx="0.00022083" ixy="0.0" ixz="0.0" iyy="0.00022083" iyz="0.0" izz="0.00040833"/>
-    </inertial>
   </link>
   <!--base_link to base_footprint Joint-->
@@ -133,4 +132,8 @@
       <material name="black"/>
     </visual>
+        <inertial>
+      <mass value="0.1"/>
+      <inertia ixx="0.00022083" ixy="0.0" ixz="0.0" iyy="0.00022083" iyz="0.0" izz="0.00040833"/>
+    </inertial>
   </link>
   <joint name="circuit_joint" type="fixed">
@@ -176,5 +179,5 @@
       </collision>
       <inertial>
-      <mass value="1"/>
+      <mass value="0.025"/>
       <inertia ixx="2.3e-06" ixy="0.0" ixz="0.0" iyy="2.3e-06" iyz="0.0" izz="4.5e-06"/>
     </inertial>
@@ -192,4 +195,45 @@
   <xacro:wheel prefix="left" reflect="1"/>
   <xacro:wheel prefix="right" reflect="-1"/>
+  <!--Tire link & joint macro-->
+  <xacro:macro name="tire" params="prefix reflect">
+    <link name="${prefix}_tire">
+      <visual>
+        <origin xyz="0 0 ${wheel_radius}" rpy="0 0 0"/>
+        <geometry>
+          <box size="0.003 ${wheel_thickness} 0.003"/>
+        </geometry>
+        <material name="darkgrey"/>
+      </visual>
+      <visual>
+        <origin xyz="0 0 ${-wheel_radius}" rpy="0 0 0"/>
+        <geometry>
+          <box size="0.003 ${wheel_thickness} 0.003"/>
+        </geometry>
+        <material name="darkgrey"/>
+      </visual>
+      <visual>
+        <origin xyz="${wheel_radius} 0 0" rpy="0 0 0"/>
+        <geometry>
+          <box size="0.003 ${wheel_thickness} 0.003"/>
+        </geometry>
+        <material name="darkgrey"/>
+      </visual>
+      <visual>
+        <origin xyz="${-wheel_radius} 0 0" rpy="0 0 0"/>
+        <geometry>
+          <box size="0.003 ${wheel_thickness} 0.003"/>
+        </geometry>
+        <material name="darkgrey"/>
+      </visual>
+    </link>
+    <joint name="${prefix}_tire_joint" type="fixed">
+      <parent link="${prefix}_wheel"/>
+      <child link="${prefix}_tire"/>
+      <origin xyz="0 0 0" rpy="0 0 0"/>
+    </joint>
+  </xacro:macro>
+  <!--Create Left & Right Wheel links/joints-->
+  <xacro:tire prefix="left" reflect="1"/>
+  <xacro:tire prefix="right" reflect="-1"/>
   <!--Motor link & joint macro-->
   <xacro:macro name="motor" params="prefix reflect">
@@ -221,14 +265,17 @@
   <link name="sensor_laser">
     <visual>
-      <geometry>
-        <box size="${laser_size_x} ${laser_size_y} ${laser_size_z}"/>
-      </geometry>
-      <material name="red"/>
-    </visual>
-    <collision>
-      <geometry>
-        <box size="${laser_size_x} ${laser_size_y} ${laser_size_z}"/>
-      </geometry>
-    </collision>
+      <origin xyz="0 0.015 0" rpy="0 ${pi/2} ${pi/3}"/>
+      <geometry>
+        <cylinder radius="${laser_size_z/2}" length="${laser_size_x*3/2}"/>
+      </geometry>
+      <material name="red"/>
+    </visual>
+    <visual>
+      <origin xyz="0 -0.015 0" rpy="0 ${pi/2} ${-pi/3}"/>
+      <geometry>
+        <cylinder radius="${laser_size_z/2}" length="${laser_size_x*3/2}"/>
+      </geometry>
+      <material name="red"/>
+    </visual>
   </link>
   <joint name="sensor_laser_joint" type="fixed">
@@ -237,4 +284,48 @@
     <child link="sensor_laser" />
   </joint>
+<!--Laser-->
+  <link name="sensor_laser_rf">
+    <visual>
+      <origin xyz="0 0 0" rpy="0 ${pi/2} 0"/>
+      <geometry>
+        <cylinder radius="${laser_size_z/2}" length="${laser_size_x}"/>
+      </geometry>
+      <material name="red"/>
+    </visual>
+    <visual>
+      <origin xyz="${laser_size_x-laser_size_z/2} 0 0" rpy="0 ${pi/2} 0"/>
+      <geometry>
+        <sphere radius="${laser_size_z/2}"/>
+      </geometry>
+      <material name="red"/>
+    </visual>
+  </link>
+  <joint name="sensor_laser_rf_joint" type="fixed">
+    <origin xyz="${wheel_joint_offset+base_len/2+(mouse_len-base_len-base_curve_radius)-laser_size_x/2} ${-(mouse_width/2-laser_size_y/2)} ${laser_origin_z}" rpy="0 0 0" />
+    <parent link="base_link"/>
+    <child link="sensor_laser_rf" />
+  </joint>
+<!--Laser-->
+  <link name="sensor_laser_lf">
+    <visual>
+      <origin xyz="0 0 0" rpy="0 ${pi/2} 0"/>
+      <geometry>
+        <cylinder radius="${laser_size_z/2}" length="${laser_size_x}"/>
+      </geometry>
+      <material name="red"/>
+    </visual>
+    <visual>
+      <origin xyz="${laser_size_x-laser_size_z/2} 0 0" rpy="0 ${pi/2} 0"/>
+      <geometry>
+        <sphere radius="${laser_size_z/2}"/>
+      </geometry>
+      <material name="red"/>
+    </visual>
+  </link>
+  <joint name="sensor_laser_lf_joint" type="fixed">
+    <origin xyz="${wheel_joint_offset+base_len/2+(mouse_len-base_len-base_curve_radius)-laser_size_x/2} ${(mouse_width/2-laser_size_y/2)} ${laser_origin_z}" rpy="0 0 0" />
+    <parent link="base_link"/>
+    <child link="sensor_laser_lf" />
+  </joint>
   <xacro:include filename="$(find micromouse_description)/urdf/mouse_gazebo.xacro"/>
 </robot>

File: micromouse_description/urdf/mouse_gazebo.xacro (robot description, xacro)
@@ -4,4 +4,10 @@
     <material>Gazebo/Red</material>
   </gazebo>
+  <gazebo reference="sensor_laser_lf">
+    <material>Gazebo/Red</material>
+  </gazebo>
+  <gazebo reference="sensor_laser_rf">
+    <material>Gazebo/Red</material>
+  </gazebo>
   <gazebo reference="front_caster_link">
     <material>Gazebo/Black</material>
@@ -23,4 +29,10 @@
               <maxVel>0.01</maxVel>
               <minDepth>0</minDepth>
+  </gazebo>
+  <gazebo reference="left_tire">
+    <material>Gazebo/DarkGrey</material>
+  </gazebo>
+  <gazebo reference="right_tire">
+    <material>Gazebo/DarkGrey</material>
   </gazebo>
   <gazebo reference="left_wheel">
@@ -78,21 +90,4 @@
               <maxVel>0.01</maxVel>
               <minDepth>0</minDepth>
-  </gazebo>
-  <gazebo reference="led">
- <material>
-            <ambient>1 0.2 0.2 1</ambient>
-            <diffuse>1 0.2 0.2 1</diffuse>
-            <specular>1 1 1 1</specular>
-            <emissive>1 0.2 0.2 1</emissive>
-          </material>
-        <light name='button' type='point'>
-          <pose>0 0 0.05 0 0 0</pose>
-          <attenuation>
-            <range>0.02</range>
-            <linear>0.10</linear>
-          </attenuation>
-          <diffuse>1 0.2 0.2 1</diffuse>
-          <specular>1 1 1 1</specular>
-        </light>
   </gazebo>
   <gazebo>
@@ -116,5 +111,5 @@
     <sensor type="ray" name="head_hokuyo_sensor">
       <pose>0 0 0 0 0 0</pose>
-      <visualize>true</visualize>
+      <visualize>false</visualize>
       <update_rate>200</update_rate>
       <ray>
@@ -144,3 +139,67 @@
     </sensor>
   </gazebo>
+<!--Gazebo Hokuyo Laser Plugin-->
+  <gazebo reference="sensor_laser_rf">
+    <sensor type="ray" name="rf_hokuyo_sensor">
+      <pose>0 0 0 0 0 0</pose>
+      <visualize>false</visualize>
+      <update_rate>200</update_rate>
+      <ray>
+        <scan>
+          <horizontal>
+            <samples>1</samples>
+            <resolution>1</resolution>
+            <min_angle>-0.1</min_angle>
+            <max_angle>-0.1</max_angle>
+          </horizontal>
+        </scan>
+        <range>
+          <min>0.01</min>
+          <max>0.25</max>
+          <resolution>0.005</resolution>
+        </range>
+        <noise>
+          <type>gaussian</type>
+          <mean>0.0</mean>
+          <stddev>0.01</stddev>
+        </noise>
+      </ray>
+      <plugin name="gazebo_ros_head_hokuyo_controller" filename="libgazebo_ros_laser.so">
+        <topicName>scanrf</topicName>
+        <frameName>sensor_laser_rf</frameName>
+      </plugin>
+    </sensor>
+  </gazebo>
+<!--Gazebo Hokuyo Laser Plugin-->
+  <gazebo reference="sensor_laser_lf">
+    <sensor type="ray" name="lf_hokuyo_sensor">
+      <pose>0 0 0 0 0 0</pose>
+      <visualize>false</visualize>
+      <update_rate>200</update_rate>
+      <ray>
+        <scan>
+          <horizontal>
+            <samples>1</samples>
+            <resolution>1</resolution>
+            <min_angle>0.1</min_angle>
+            <max_angle>0.1</max_angle>
+          </horizontal>
+        </scan>
+        <range>
+          <min>0.01</min>
+          <max>0.25</max>
+          <resolution>0.005</resolution>
+        </range>
+        <noise>
+          <type>gaussian</type>
+          <mean>0.0</mean>
+          <stddev>0.01</stddev>
+        </noise>
+      </ray>
+      <plugin name="gazebo_ros_head_hokuyo_controller" filename="libgazebo_ros_laser.so">
+        <topicName>scanlf</topicName>
+        <frameName>sensor_laser_lf</frameName>
+      </plugin>
+    </sensor>
+  </gazebo>
 </robot>
